Commit message: 수확 로봇 관련 commit

File: dsr_description/xacro/m0609.urdf.xacro (robot description, xacro)
@@ -7,4 +7,7 @@
   <xacro:if value="${cr == 'white'}">
      <xacro:include filename="$(find dsr_description)/xacro/macro.m0609.white.xacro" />
+     <xacro:include filename="$(find realsense2_description)/urdf/_d435.urdf.xacro" />
+     <xacro:include filename="$(find dsr_description)/xacro/cwsfa_mobilebase.xacro" />
+     <xacro:include filename="$(find dsr_description)/xacro/cucumber_gripper.xacro" />
   </xacro:if>
   <xacro:if value="${cr == 'blue'}">
@@ -12,13 +15,29 @@
   </xacro:if>
   <xacro:m0609 namespace="$(arg namespace)"/>
-  <link name="world" />
   <xacro:if value="${gr == 'robotiq_2f'}">
      <xacro:include filename="$(find dsr_description)/xacro/robotiq_2f.urdf.xacro" />
   </xacro:if>
   <!-- World fixed joint-->
+  <link name="world" />
   <joint name="world_fixed" type="fixed">
-    <origin xyz="0 0 0" rpy="0 0 0"/>
+    <origin xyz="0 0 0.35" rpy="0 0 0"/>
     <parent link="world"/>
+    <child link="mobile_base"/>
+  </joint>
+  <!-- cw_mobilebase with M0609 -->
+  <joint name="m0609_fixed" type="fixed">
+    <origin xyz="0.07 0.13 0.35" rpy="0 0 0"/>
+    <parent link="mobile_base"/>
     <child link="base_0"/>
   </joint>
+  <!-- cucumber_gripper with J6 -->
+  <joint name="grip_joint" type="fixed">
+    <origin xyz="0.0 0.019 0.181" rpy="0 0 0"/>
+    <parent link="link6"/>
+    <child link="gripper"/>
+  </joint>
+  <sensor_d435 parent="link6">
+    <!-- Link6 standard: Y, -Z, X -->
+    <origin xyz="0 -0.0785 0.03815" rpy="0 -1.5707 1.5707"/>
+  </sensor_d435>
 </robot>
